Commit message: Get cart example to work
Signed-off-by: Yadunund <yadunund@intrinsic.ai>

File: mujoco_ros2_control_demos/urdf/test_cart_effort.xacro.urdf (robot description, URDF)
Before this commit: robot cartopole, 4 links, 3 joints
Links:
- removed link cart_imu
Joints:
- removed joint cart_to_imu
